Commit message: Add simulation of task1

File: src/rascl_description/urdf/rascl.urdf (robot description, URDF)
Before this commit: robot rascl_bot, 6 links, 5 joints
Joints:
- joint lowerarm_joint: origin xyz=0.17 0.08 0.02183 rpy=0 3.14159265 0 -> xyz=0.17 0.08 0.02183 rpy=0 3.14159265 -1.570796327

Commit message: update setup and urdf

File: src/rascl_description/urdf/rascl.urdf (robot description, URDF)
Before this commit: robot rascl_bot, 6 links, 5 joints
Joints:
- joint lowerarm_joint: axis 0 0 1 -> 0 0 -1
- joint shoulder_joint: axis 0 0 1 -> 0 0 -1
- joint upperarm_joint: axis 0 0 1 -> 0 0 -1
